Commit message: updated with custom map and world

File: remote/urdf/turtlebot3_waffle.urdf (robot description, URDF)
Before this commit: robot turtlebot3_waffle, 13 links, 12 joints
Links:
- link base_link: geometry collision box size=0.266 0.266 0.094; visual mesh filename=package://urdf/meshes/chassis.stl scale=0.001 0.001 0.001
